File: espbb.sch (KiCad schematic (older format))
At the start: 9 parts, among them P1 CONN_8, P2 CONN_8, SW1 SWITCH_INV, U1 ESP-12/07V2/08V2, U2 LM6206

Commit message: esp-12e version
Parts:
- removed P1, P2: CONN_8, symbol CONN_8
- removed U1: ESP-12/07V2/08V2, ~, symbol ESP-12/07V2/08V2
- added P1, P2: CONN_01X12, Pin_Headers:Pin_Header_Straight_1x12, symbol CONN_01X12
- added R3: 0Ohm, r0603:SM0603, symbol R-RESCUE-espbb
- added U1: ESP-12E, esp8266:ESP-12E, symbol ESP-12E
- added U3: AMS1117-3.3, sot223:SOT223, symbol LM6206
- C1, C2: footprint ~ -> Capacitors_SMD:C_0603; symbol C -> C-RESCUE-espbb
- R1, R2: footprint ~ -> r0603:SM0603; symbol R -> R-RESCUE-espbb
- SW1: footprint ~ -> jumperswitch:SIL-3
Connections:
- wire segments 48 -> 83
